Commit message: planner: link boxes on robot links; base, quaternion and wrist-adjacency fixes; URDF boxes re-fitted
- link_boxes: a box that belongs to a robot link (a camera on the wrist,
  a bracket on the forearm), pose in that link's frame — Planner.update(
  link_boxes={link: [cube]}), plan/check_path(link_boxes=[{link, pose,
  scale, type}]); C++ InputLinkShape + attachLinkShapes adds it to the
  link's own geometry (moves with it, hits the world and non-adjacent
  links, never its own link or neighbours); an unknown link name raises
- has_camera and dorna_ta_camera.urdf are gone: one URDF, the camera is
  a link box the workspace passes
- Planner.link_frames(joint, base_in_world) and robot_boxes(joint,
  base_in_world): the links' world frames and URDF boxes as the planner
  places them; stored tool / base / frame keep their mm copies, so a
  subset update() no longer rescales them each rebuild
- node.py: python-fcl Transform takes [w, x, y, z]; every rotated box the
  python checker built was mis-oriented (a 90 deg turn rendered as a
  180 deg flip); robot links were unaffected (rotation matrices)
- planner.hpp: the load / gripper is not tested against the adjacent
  wrist link, the same parent/child rule the links use (a tool box
  touching the wrist invalidated every pose)
- urdf/dorna_ta.urdf: the 14 link boxes re-fitted to the link meshes by
  tools/refit_urdf_boxes.py (margin 0, base boxes 1 mm above the
  mounting plane); same count and orientation, rerun when a mesh changes

Co-Authored-By: Claude Fable 5.1 <noreply@anthropic.com>

File: resources/urdf/dorna_ta.urdf (robot description, URDF)
Before this commit: robot DornaTA, 7 links, 6 joints
Links:
- link j0_link: geometry collision box size=0.181201 0.116002 0.007000; collision box size=0.187200 0.086403 0.117007
- link j1_link: geometry collision box size=0.057423 0.059173 0.057423; collision box size=0.203320 0.078001 0.090444
- link j2_link: geometry collision box size=0.057077 0.057187 0.046383; collision box size=0.301200 0.066406 0.065007
- link j3_link: geometry collision box size=0.039008 0.042402 0.042402; collision box size=0.054001 0.101200 0.062403
- link j4_link: geometry collision box size=0.042398 0.039000 0.042398; collision box size=0.043003 0.000000 0.006001
- link j5_link: geometry collision box size=0.047313 0.042321 0.037002; collision box size=0.088200 0.046403 0.056000
- link j6_link: geometry collision box size=0.043000 0.006000 0.042879
